Commit message: Add mast for camera.

File: leo_description/urdf/ld06_lidar_mount.urdf.xacro (robot description, xacro)
@@ -9,5 +9,5 @@
                 <origin xyz="0.0 0.0 0.0" rpy="0 0 0"/>
                 <geometry>
-                    <mesh filename="package://leo_description/models/ld06_lidar_msm_assembly_coloured.dae"/>
+                    <mesh filename="package://leo_description/models/model_extensions/ld06_lidar_msm_assembly_coloured.dae"/>
                 </geometry>
                 <geometry>

File: leo_description/urdf/leo.urdf.xacro (robot description, xacro)
@@ -4,6 +4,8 @@
   <xacro:arg name="mecanum_wheels" default="false"/>
   <xacro:include filename="$(find leo_description)/urdf/macros.xacro"/>
+  <xacro:include filename="$(find leo_description)/urdf/mast.xacro"/>
   <xacro:include filename="$(find leo_description)/urdf/ld06_lidar_mount.urdf.xacro"/>
   <xacro:leo mecanum_wheels="$(arg mecanum_wheels)"/>
   <xacro:ld06_lidar_module/>
+  <xacro:leo_mast/>
 </robot>

Commit message: Add realsense camera and xavier.

File: leo_description/urdf/ld06_lidar_mount.urdf.xacro (robot description, xacro)
@@ -10,7 +10,4 @@
                 <geometry>
                     <mesh filename="package://leo_description/models/model_extensions/ld06_lidar_msm_assembly_coloured.dae"/>
-                </geometry>
-                <geometry>
-                    <cylinder length="0.2" radius="0.025"/>
                 </geometry>
             </visual>

File: leo_description/urdf/leo.urdf.xacro (robot description, xacro)
@@ -3,4 +3,5 @@
        name="leo">
   <xacro:arg name="mecanum_wheels" default="false"/>
+  <xacro:arg name="d455_camera" default="true"/>
   <xacro:include filename="$(find leo_description)/urdf/macros.xacro"/>
   <xacro:include filename="$(find leo_description)/urdf/mast.xacro"/>

File: leo_description/urdf/mast.xacro (robot description, xacro)
@@ -3,4 +3,5 @@
   <xacro:macro name="leo_mast"
                params="default_mikrotik_antenna:=true
+                       d455_camera:=true
                        link_prefix:=''
                        joint_prefix:=''">
@@ -94,4 +95,16 @@
     </joint>
   </xacro:if>
+  <xacro:if value="${d455_camera}">
+    <link name="${link_prefix}realsense_link"/>
+    <xacro:include filename="$(find realsense2_description)/urdf/_d455.urdf.xacro"/>
+    <xacro:sensor_d455 name="${link_prefix}realsense_camera" parent="${link_prefix}realsense_link">
+      <origin xyz="0.0 0.0 0.0" rpy="0 0 0"/>
+    </xacro:sensor_d455>
+    <joint name="${link_prefix}realsense_joint" type="fixed">
+      <origin xyz="0.0 0 0.0" rpy="0 0 0"/>
+      <parent link="${link_prefix}mast_camera_screw_frame"/>
+      <child link="${link_prefix}realsense_link"/>
+    </joint>
+  </xacro:if>
   </xacro:macro>
 </robot>
