Commit message: Clean up.

File: leo_description/urdf/xavier_mount.xacro (robot description, xacro)
@@ -93,5 +93,5 @@
   </link>
   <joint name="${joint_prefix}makita_battery_joint" type="fixed">
-    <origin xyz="0.005 0.0 0.025" rpy="0 0 0"/>
+    <origin xyz=" 0.005 0.0 0.025" rpy="0 0 0"/>
     <parent link="${link_prefix}makita_battery_adapter"/>
     <child link="${link_prefix}makita_battery"/>
