Commit message: Add battery and xavier to URDF.

File: leo_description/urdf/leo.urdf.xacro (robot description, xacro)
@@ -7,6 +7,8 @@
   <xacro:include filename="$(find leo_description)/urdf/mast.xacro"/>
   <xacro:include filename="$(find leo_description)/urdf/ld06_lidar_mount.urdf.xacro"/>
+  <xacro:include filename="$(find leo_description)/urdf/xavier_mount.xacro"/>
   <xacro:leo mecanum_wheels="$(arg mecanum_wheels)"/>
   <xacro:ld06_lidar_module/>
   <xacro:leo_mast/>
+  <xacro:xavier_mount/>
 </robot>

File: leo_description/urdf/xavier_mount.xacro (robot description, xacro)
@@ -7,7 +7,7 @@
   <link name="${link_prefix}makita_battery_mount">
     <visual>
-    <origin xyz="0.0 0.0 0.0" rpy="0 0 0"/><!-- ${-pi/2} -->
+    <origin xyz="0.0 0.0 0.0" rpy="0 0 0"/>
       <geometry>
-        <mesh filename="package://leorover_description/models/model_extensions/makita_battery_mount.dae"/>
+        <mesh filename="package://leo_description/models/model_extensions/makita_battery_mount.dae"/>
       </geometry>
     </visual>
@@ -40,5 +40,5 @@
     <origin xyz="0.0 0.0 0.0" rpy="0 0 0"/>
       <geometry>
-        <mesh filename="package://leorover_description/models/model_extensions/makita_battery_adapter.dae"/>
+        <mesh filename="package://leo_description/models/model_extensions/makita_t_mount_M3.dae"/>
       </geometry>
     </visual>
@@ -62,5 +62,5 @@
   </link>
   <joint name="${joint_prefix}makita_battery_adapter_joint" type="fixed">
-    <origin xyz="0.0 0.0 0.015" rpy="0 0 0"/>
+    <origin xyz="-0.01 0.0 0.015" rpy="0 0 0"/>
     <parent link="${link_prefix}makita_battery_mount"/>
     <child link="${link_prefix}makita_battery_adapter"/>
@@ -71,5 +71,5 @@
     <origin xyz="0.0 0.0 0.035" rpy="0 ${pi} 0"/>
       <geometry>
-        <mesh filename="package://leorover_description/models/model_extensions/makita_battery.dae"/>
+        <mesh filename="package://leo_description/models/model_extensions/makita_battery.dae"/>
       </geometry>
     </visual>
@@ -93,5 +93,5 @@
   </link>
   <joint name="${joint_prefix}makita_battery_joint" type="fixed">
-    <origin xyz="-0.005 0.0 0.035" rpy="0 0 0"/>
+    <origin xyz="0.005 0.0 0.025" rpy="0 0 0"/>
     <parent link="${link_prefix}makita_battery_adapter"/>
     <child link="${link_prefix}makita_battery"/>
@@ -100,7 +100,7 @@
   <link name="${link_prefix}xavier_mount">
     <visual>
-    <origin xyz="0.0 0.0 0.0" rpy="0 0 0"/><!-- ${-pi/2} -->
+    <origin xyz="0.0 0.0 0.0" rpy="0 0 0"/>
       <geometry>
-        <mesh filename="package://leorover_description/models/model_extensions/xavier_mount.dae"/>
+        <mesh filename="package://leo_description/models/model_extensions/xavier_mount.dae"/>
       </geometry>
     </visual>

Commit message: Add lidar position as calibrated lidar

File: leo_description/urdf/leo.urdf.xacro (robot description, xacro)
@@ -4,19 +4,19 @@
   <xacro:arg name="mecanum_wheels" default="false"/>
   <!-- <xacro:arg name="d455_camera" default="true"/> -->
-  <xacro:arg name="zed2_camera" default="false"/>
+  <!-- <xacro:arg name="zed2_camera" default="false"/>
   <xacro:arg name="zed2_camera_model" default="true"/>
   <xacro:arg name="optitrack_marker_link" default="true"/>
-  <xacro:arg name="livox_hap_model" default="true"/>
+  <xacro:arg name="livox_hap_model" default="true"/> -->
   <xacro:include filename="$(find leo_description)/urdf/macros.xacro"/>
   <!-- <xacro:include filename="$(find leo_description)/urdf/mast.xacro"/> -->
   <!-- <xacro:include filename="$(find leo_description)/urdf/ld06_lidar_mount.urdf.xacro"/> -->
   <!-- <xacro:include filename="$(find leo_description)/urdf/xavier_mount.xacro"/> -->
-  <xacro:include filename="$(find leo_description)/urdf/leorover_backpack.xacro"/>
-  <xacro:include filename="$(find leo_description)/urdf/leorover_frontpack.xacro"/>
+  <!-- <xacro:include filename="$(find leo_description)/urdf/leorover_backpack.xacro"/>
+  <xacro:include filename="$(find leo_description)/urdf/leorover_frontpack.xacro"/> -->
   <xacro:leo mecanum_wheels="$(arg mecanum_wheels)"/>
   <!-- <xacro:ld06_lidar_module/> -->
   <!-- <xacro:leo_mast/> -->
   <!-- <xacro:xavier_mount/> -->
-  <xacro:leorover_backpack/>
-  <xacro:leorover_frontpack/>
+  <!-- <xacro:leorover_backpack/>
+  <xacro:leorover_frontpack/> -->
 </robot>

File: leo_description/urdf/leorover_frontpack.xacro (robot description, xacro)
@@ -1,119 +1,132 @@
 <?xml version="1.0" encoding="utf-8"?>
 <robot xmlns:xacro="http://www.ros.org/wiki/xacro">
-<xacro:macro name="leorover_frontpack"
-               params="zed2_camera:=false
-                        zed2_camera_model:=true
-                        optitrack_marker_link:=true
-                        livox_hap_model:=true
-                        link_prefix:=''
-                        joint_prefix:=''">
- <link name="${link_prefix}frontpack_link">
-        <inertial>
-            <mass value="1.0"/>
-            <inertia
-            ixx="0.00905" ixy="0.0" ixz="0.0"
-            iyy="0.00545"  iyz="0.0"
-            izz="0.00850"/>
-        </inertial>
-        <visual>
-            <origin xyz="0 0 0" rpy="0 0 0"/>
-            <geometry>
-                <mesh filename="package://leo_description/models/model_extensions/leorover_frontpack.dae"/>
-            </geometry>
-        </visual>
-        <collision>
-            <origin xyz="0.0 0.0 0.10"/>
-            <geometry>
-                <box size="0.14 0.18 0.20"/>
-            </geometry>
-        </collision>
-        <collision>
-            <origin xyz="0.04 0.0 0.265"/>
-            <geometry>
-                <box size="0.07 0.11 0.13"/>
-            </geometry>
-        </collision>
-    </link>
-    <joint name="${joint_prefix}leorover_frontpack_joint" type="fixed">
-        <origin xyz="0.067 0.0 0.0" rpy="0 0 0"/>
-        <parent link="${link_prefix}base_link"/>
-        <child link="${link_prefix}frontpack_link"/>
-    </joint>
-    <!-- Placeholder for the camera screw at the camera mount position (25 degrees) not rotated. -->
-    <link name="${link_prefix}camera_mount_screw_link"/>
-    <joint name="${joint_prefix}camera_mount_screw_joint" type="fixed">
-        <origin xyz="0.044557 0.0 0.25876" rpy="0 0 0"/>
-        <parent link="${link_prefix}frontpack_link"/>
-        <child link="${link_prefix}camera_mount_screw_link"/>
-    </joint>
-    <xacro:if value="${zed2_camera}">
-    <!-- {name}_camera_link -->
-        <joint name="${joint_prefix}_camera_link_joint" type="fixed">
-            <origin xyz="0.0 0.0 0.0" rpy="0 0.4363 0"/>
-            <parent link="${link_prefix}camera_mount_screw_link"/>
-            <child link="${link_prefix}zed2_camera_link"/>
+    <xacro:macro name="leorover_frontpack"
+                params="zed2_camera:=false
+                            zed2_camera_model:=true
+                            optitrack_marker_link:=true
+                            livox_hap_model:=true
+                            link_prefix:=''
+                            joint_prefix:=''">
+        <link name="${link_prefix}frontpack_link">
+            <inertial>
+                <mass value="1.0"/>
+                <inertia
+                    ixx="0.00905" ixy="0.0" ixz="0.0"
+                    iyy="0.00545"  iyz="0.0"
+                    izz="0.00850"/>
+            </inertial>
+            <visual>
+                <origin xyz="0 0 0" rpy="0 0 0"/>
+                <geometry>
+                    <mesh filename="package://leo_description/models/model_extensions/leorover_frontpack.dae"/>
+                </geometry>
+            </visual>
+            <collision>
+                <origin xyz="0.0 0.0 0.10"/>
+                <geometry>
+                    <box size="0.14 0.18 0.20"/>
+                </geometry>
+            </collision>
+            <collision>
+                <origin xyz="0.04 0.0 0.265"/>
+                <geometry>
+                    <box size="0.07 0.11 0.13"/>
+                </geometry>
+            </collision>
+        </link>
+        <joint name="${joint_prefix}leorover_frontpack_joint" type="fixed">
+            <origin xyz="0.067 0.0 0.0" rpy="0 0 0"/>
+            <parent link="${link_prefix}base_link"/>
+            <child link="${link_prefix}frontpack_link"/>
         </joint>
-        <link name="${link_prefix}zed2_camera_link"/>
-    </xacro:if>
-    <xacro:if value="${zed2_camera_model}">
-    <!-- {name}_camera_link -->
-        <joint name="${joint_prefix}_camera_link_joint" type="fixed">
-            <origin xyz="0.0 0.0 0.0" rpy="0 0.4363 0"/>
-            <parent link="${link_prefix}camera_mount_screw_link"/>
-            <child link="${link_prefix}zed2_camera_link"/>
+        <!-- Placeholder for the camera screw at the camera mount position (25 degrees) not rotated. -->
+        <link name="${link_prefix}camera_mount_screw_link"/>
+        <joint name="${joint_prefix}camera_mount_screw_joint" type="fixed">
+            <origin xyz="0.044557 0.0 0.25876" rpy="0 0 0"/>
+            <parent link="${link_prefix}frontpack_link"/>
+            <child link="${link_prefix}camera_mount_screw_link"/>
         </joint>
-        <link name="${link_prefix}zed2_camera_link">
-        <inertial>
-            <mass value="0.3"/>
-            <inertia
-            ixx="0.0008325" ixy="0.0" ixz="0.0"
-            iyy="0.0000625"  iyz="0.0"
-            izz="0.00085"/>
-        </inertial>
-        <visual>
-            <origin xyz="0 0 0" rpy="0 0 0"/>
-            <geometry>
-                <mesh filename="package://leo_description/models/model_extensions/zed2_camera.dae"/>
-            </geometry>
-        </visual>
-        <collision>
-            <origin xyz="0.0 0.0 0.015"/>
-            <geometry>
-                <box size="0.04 0.18 0.03"/>
-            </geometry>
-        </collision>
-    </link>
-    </xacro:if>
-    <xacro:if value="${optitrack_marker_link}">
-        <joint name="${joint_prefix}_optitrack_marker_joint" type="fixed">
-            <origin xyz="0.009 0.0 0.053" rpy="0 0.468 0"/>
-            <parent link="${link_prefix}camera_mount_screw_link"/>
-            <child link="${link_prefix}optitrack_marker_link:"/>
-        </joint>
-        <link name="${link_prefix}optitrack_marker_link:">
-        <visual>
-            <origin xyz="0 0 0" rpy="0 0 0"/>
-            <geometry>
-                <mesh filename="package://leo_description/models/model_extensions/optitrack_marker.dae"/>
-            </geometry>
-        </visual>
-    </link>
-    </xacro:if>
-        <xacro:if value="${livox_hap_model}">
-    <!-- {name}_camera_link -->
-        <joint name="${joint_prefix}_livox_hap_model_link_joint" type="fixed">
-            <origin xyz="0.009 0.0 0.1035" rpy="0 0 0"/>
-            <parent link="${link_prefix}frontpack_link"/>
-            <child link="${link_prefix}livox_hap_model_link"/>
-        </joint>
-        <link name="${link_prefix}livox_hap_model_link">
-        <visual>
-            <origin xyz="0 0 0" rpy="0 0 0"/>
-            <geometry>
-                <mesh filename="package://leo_description/models/model_extensions/livox_hap_model.dae"/>
-            </geometry>
-        </visual>
-    </link>
-    </xacro:if>
-  </xacro:macro>
+        <xacro:if value="${zed2_camera}">
+            <!-- {name}_camera_link -->
+            <joint name="${joint_prefix}_camera_link_joint" type="fixed">
+                <origin xyz="0.0 0.0 0.0" rpy="0 0.4363 0"/>
+                <parent link="${link_prefix}camera_mount_screw_link"/>
+                <child link="$zed2_camera_link"/>
+            </joint>
+            <link name="zed2_camera_link"/>
+        </xacro:if>
+        <xacro:if value="${zed2_camera_model}">
+            <!-- {name}_camera_link -->
+            <joint name="${joint_prefix}_camera_link_joint" type="fixed">
+                <origin xyz="0.0 0.0 0.0" rpy="0 0.4363 0"/>
+                <parent link="${link_prefix}camera_mount_screw_link"/>
+                <child link="zed2_camera_link"/>
+            </joint>
+            <link name="zed2_camera_link">
+            <inertial>
+                <mass value="0.3"/>
+                <inertia
+                    ixx="0.0008325" ixy="0.0" ixz="0.0"
+                    iyy="0.0000625"  iyz="0.0"
+                    izz="0.00085"/>
+                </inertial>
+            <visual>
+                <origin xyz="0 0 0" rpy="0 0 0"/>
+                <geometry>
+                    <mesh filename="package://leo_description/models/model_extensions/zed2_camera.dae"/>
+                </geometry>
+            </visual>
+            <collision>
+                <origin xyz="0.0 0.0 0.015"/>
+                <geometry>
+                    <box size="0.04 0.18 0.03"/>
+                </geometry>
+            </collision>
+        </link>
+        </xacro:if>
+        <xacro:if value="${optitrack_marker_link}">
+            <joint name="${joint_prefix}_optitrack_marker_joint" type="fixed">
+                <origin xyz="0.009 0.0 0.053" rpy="0 0.468 0"/>
+                <parent link="${link_prefix}camera_mount_screw_link"/>
+                <child link="${link_prefix}optitrack_marker_link"/>
+            </joint>
+            <link name="${link_prefix}optitrack_marker_link">
+                <visual>
+                    <origin xyz="0 0 0" rpy="0 0 0"/>
+                    <geometry>
+                        <mesh filename="package://leo_description/models/model_extensions/optitrack_marker.dae"/>
+                    </geometry>
+                </visual>
+            </link>
+        </xacro:if>
+            <xacro:if value="${livox_hap_model}">
+            <!-- {name}_camera_link -->
+            <joint name="${joint_prefix}_livox_hap_model_link_joint" type="fixed">
+                <origin xyz="0.009 0.0 0.1035" rpy="0 0 0"/>
+                <parent link="${link_prefix}frontpack_link"/>
+                <child link="${link_prefix}livox_hap_model_link"/>
+            </joint>
+            <link name="${link_prefix}livox_hap_model_link">
+                <visual>
+                    <origin xyz="0 0 0" rpy="0 0 0"/>
+                    <geometry>
+                        <mesh filename="package://leo_description/models/model_extensions/livox_hap_model.dae"/>
+                    </geometry>
+                </visual>
+            </link>
+            <link name="${link_prefix}livox_frame"/>
+            <!-- Position derived from datasheet -->
+	    <!-- <joint name="${joint_prefix}livox_frame_joint" type="fixed"> -->
+	    <!-- <origin xyz="0.04775 0.0 0.023" rpy="0 0 0"/> -->
+	    <!-- <parent link="${link_prefix}livox_hap_model_link"/> -->
+	    <!-- <child link="${link_prefix}livox_frame"/> -->
+	    <!-- </joint> -->
+	    <!-- Position derived from calibration -->
+            <joint name="${joint_prefix}livox_frame_joint" type="fixed">
+                <origin xyz="0.015 0.005 0.030" rpy="0.001 0.016 -0.041"/>
+                <parent link="${link_prefix}livox_hap_model_link"/>
+                <child link="${link_prefix}livox_frame"/>
+            </joint>
+        </xacro:if>
+    </xacro:macro>
 </robot>
